File: ExternalPower.sch (KiCad schematic (older format))
At the start: 6 parts, among them J1 GS3

Commit message: feat: alignment
Connections:
- net Ground renamed GND
Changed lines of the file:
@@
 Wire Wire Line
 	6170 4730 6170 4290
-Text HLabel 6685 4730 2    60   Input ~ 0
-Ground
+Text HLabel 6685 4730 2    39   Input ~ 0
+GND
 Connection ~ 6170 4730
-Text HLabel 6685 3570 2    60   Input ~ 0
+Text HLabel 6685 3570 2    39   Input ~ 0
 VIN
 Connection ~ 6170 3570
-Text HLabel 4665 3025 0    60   Input ~ 0
+Text HLabel 4665 3025 0    39   Input ~ 0
 12V
-Text HLabel 5270 3025 2    60   Input ~ 0
+Text HLabel 5270 3025 2    39   Input ~ 0
 5.5V
 Wire Wire Line
