File: MAX7480Block.sch (KiCad schematic (older format))
At the start: 8 parts

Commit message: feat: RC block 2
Parts:
- gave numbers to parts that had none: 8
Changed lines of the file:
@@
 $Descr A4 11693 8268
 encoding utf-8
-Sheet 6 6
+Sheet 6 8
 Title ""
 Date ""
@@
 $EndDescr
 $Comp
-L MAX7480ESA+ U?
+L MAX7480ESA+ U5
 U 1 1 5B10B68A
 P 4770 3365
-F 0 "U?" H 4770 3115 39  0000 C CNN
+F 0 "U5" H 4770 3115 39  0000 C CNN
 F 1 "MAX7480ESA+" H 4820 3615 39  0000 C CNN
 F 2 "" H 4820 3265 30  0001 C CNN
@@
 $EndComp
 $Comp
-L MAX7480ESA+ U?
+L MAX7480ESA+ U6
 U 1 1 5B10B6BF
 P 4775 4495
-F 0 "U?" H 4775 4245 39  0000 C CNN
+F 0 "U6" H 4775 4245 39  0000 C CNN
 F 1 "MAX7480ESA+" H 4825 4745 39  0000 C CNN
 F 2 "" H 4825 4395 30  0001 C CNN
@@
 $EndComp
 $Comp
-L MAX7480ESA+ U?
+L MAX7480ESA+ U7
 U 1 1 5B10BE2A
 P 7215 3365
-F 0 "U?" H 7215 3115 39  0000 C CNN
+F 0 "U7" H 7215 3115 39  0000 C CNN
 F 1 "MAX7480ESA+" H 7265 3615 39  0000 C CNN
 F 2 "" H 7265 3265 30  0001 C CNN
@@
 $EndComp
 $Comp
-L MAX7480ESA+ U?
+L MAX7480ESA+ U8
 U 1 1 5B10BE30
 P 7220 4495
-F 0 "U?" H 7220 4245 39  0000 C CNN
+F 0 "U8" H 7220 4245 39  0000 C CNN
 F 1 "MAX7480ESA+" H 7270 4745 39  0000 C CNN
 F 2 "" H 7270 4395 30  0001 C CNN
@@
 OUT4
 $Comp
-L C C?
+L C C14
 U 1 1 5B10D3B0
 P 3470 3215
-F 0 "C?" H 3495 3315 50  0000 L CNN
+F 0 "C14" H 3495 3315 50  0000 L CNN
 F 1 "0.1u" H 3495 3115 50  0000 L CNN
 F 2 "" H 3508 3065 50  0001 C CNN
@@
 $EndComp
 $Comp
-L C C?
+L C C15
 U 1 1 5B10D6EE
 P 3470 4365
-F 0 "C?" H 3495 4465 50  0000 L CNN
+F 0 "C15" H 3495 4465 50  0000 L CNN
 F 1 "0.1u" H 3495 4265 50  0000 L CNN
 F 2 "" H 3508 4215 50  0001 C CNN
@@
 $EndComp
 $Comp
-L C C?
+L C C16
 U 1 1 5B10DFB3
 P 6075 3240
-F 0 "C?" H 6100 3340 39  0000 L CNN
+F 0 "C16" H 6100 3340 39  0000 L CNN
 F 1 "0.1u" H 6100 3140 39  0000 L CNN
 F 2 "" H 6113 3090 50  0001 C CNN
@@
 $EndComp
 $Comp
-L C C?
+L C C17
 U 1 1 5B10EAFE
 P 6075 4365
-F 0 "C?" H 6100 4465 39  0000 L CNN
+F 0 "C17" H 6100 4465 39  0000 L CNN
 F 1 "0.1u" H 6100 4265 39  0000 L CNN
 F 2 "" H 6113 4215 50  0001 C CNN

Commit message: feat: alignment
Changed lines of the file:
@@
 encoding utf-8
 Sheet 6 10
-Title ""
-Date ""
-Rev ""
+Title "FOSSASIA - NeuroFox"
+Date "2018-05-31"
+Rev "1"
 Comp ""
 Comment1 ""
@@
 	5270 3315 5720 3315
 Wire Wire Line
-	5720 3045 5720 3315
-Wire Wire Line
-	3470 3045 5720 3045
+	5720 3315 5720 3045
+Wire Wire Line
+	5720 3045 3470 3045
 Wire Wire Line
 	4225 3045 4225 3215
@@
 	5275 4445 5740 4445
 Wire Wire Line
-	5740 4180 5740 4445
-Wire Wire Line
-	3470 4180 5740 4180
+	5740 4445 5740 4180
+Wire Wire Line
+	5740 4180 3470 4180
 Wire Wire Line
 	4225 4180 4225 4345
@@
 	7720 4445 8245 4445
 Wire Wire Line
-	8245 4190 8245 4445
-Wire Wire Line
-	6075 4190 8245 4190
+	8245 4445 8245 4190
+Wire Wire Line
+	8245 4190 6075 4190
 Wire Wire Line
 	6660 4190 6660 4345
@@
 	7715 3315 8240 3315
 Wire Wire Line
-	8240 3060 8240 3315
-Wire Wire Line
-	6075 3060 8240 3060
+	8240 3315 8240 3060
+Wire Wire Line
+	8240 3060 6075 3060
 Wire Wire Line
 	6660 3060 6660 3215
